File: designs/beeper-flex/kicad/beeper-flex.kicad_sch (KiCad schematic)
At the start: 5 parts, among them U3 IM69D130V01XTSA1, U4 IM69D130V01XTSA1, U6 Edge-FH19C-4S-0.5SH(10)

Commit message: somewhat stable flex design
Parts:
- removed U6: Edge-FH19C-4S-0.5SH(10), beeper-flex:EDGE_LP, symbol edge_FH19C_4S_0_5SH_10_
- added U6: Edge-FH19C-6S-0.5SH(10), beeper-flex:EDGE_LP, symbol edge_FH19C_6S_0_5SH_10_
Connections:
- net GND: now also U6.2, U6.3, U6.4
- net PDM_clk: now also U6.1
- net PDM_data: now also U6.5
- net VDDMIC: now also U6.6
