File: designs/beeper-flex/kicad/beeper-flex.kicad_pcb (KiCad board)
At the start: 2 copper layers, 22.2 x 7.9 mm, 7 parts

Commit message: updated gerbers for flex
Other:
- rule pad_to_mask_clearance: 0.051 -> 0
Changed lines of the file:
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@@
       (dielectric_constraints no)
     )
-    (pad_to_mask_clearance 0.051)
+    (pad_to_mask_clearance 0)
     (pcbplotparams
-      (layerselection 0x0000030_80000001)
-      (plot_on_all_layers_selection 0x0000000_00000000)
+      (layerselection 0x00012fc_ffffffff)
+      (plot_on_all_layers_selection 0x0001000_00000000)
       (disableapertmacros false)
       (usegerberextensions false)
@@
       (outputformat 1)
       (mirror false)
-      (drillshape 1)
+      (drillshape 0)
       (scaleselection 1)
-      (outputdirectory "")
+      (outputdirectory "gerbers/")
     )
   )
