File: designs/beeper-design/kicad/beeper-design.kicad_pcb (KiCad board)
At the start: 4 copper layers, 27.5 x 19 mm, 99 parts

Commit message: updated kicad export
Parts:
- removed the C14 at (147.0, 103.3)
- removed the C23 at (148.3, 99.4)
- removed the C4 at (145.6, 109.9)
- removed the R10 at (133.2, 109.8)
- removed the R15 at (133.1, 109.1)
- removed the R4 at (144.5, 100.1)
- removed the R7 at (145.3, 99.6)
- removed the U15 at (137.8, 106.8)
- removed the U5 at (148.8, 113.7)
- added C20: 10n, beeper-design:Pkg0201_30, F.Cu at (149.3, 99.8)
- added C43: 100n, beeper-design:Pkg0201_39, F.Cu at (129.3, 108.6)
- added C6: 47u, beeper-design:Pkg0805_1, F.Cu at (145.6, 112.4)
- added J1: ~, beeper-design:TC2030_IDC_NL_FOOTPRINT, B.Cu at (129.7, 102.5)
- added J6: ~, beeper-design:AMPHENOL_10103594_0001LF, B.Cu at (137.1, 100.5)
- added L4: 1n, beeper-design:Pkg0201_41, F.Cu at (131.2, 116.0)
- added R16: 8K2, beeper-design:Pkg0201_20, F.Cu at (134.6, 106.2)
- added U2: ~, beeper-design:WLCSP_12, F.Cu at (144.2, 115.5)
- added U3: ~, beeper-design:LP_7, F.Cu at (147.0, 101.5)
- C14: renamed from R5; value 10K -> 2.2u; footprint beeper-design:Pkg0201_22 -> beeper-design:Pkg0201_25
- C23: renamed from J6; value ~ -> 10u; footprint beeper-design:AMPHENOL_10103594_0001LF -> beeper-design:Pkg0402_2; moved to F.Cu
- C4: renamed from U3; value ~ -> 47u; footprint beeper-design:LP_7 -> beeper-design:Pkg0805
- R10: renamed from R3; value 196R -> 0R; footprint beeper-design:Pkg0201_2 -> beeper-design:Pkg0201_28
- R15: renamed from J1; value ~ -> 8K2; footprint beeper-design:TC2030_IDC_NL_FOOTPRINT -> beeper-design:Pkg0201_1; moved to F.Cu
- R3: renamed from L4; value 1n -> 196R; footprint beeper-design:Pkg0201_41 -> beeper-design:Pkg0201_2
- R4: renamed from C6; value 47u -> 20K; footprint beeper-design:Pkg0805_1 -> beeper-design:Pkg0201_12
- R5: renamed from R16; value 8K2 -> 10K; footprint beeper-design:Pkg0201_20 -> beeper-design:Pkg0201_22
- R7: renamed from U9; value ~ -> 10K; footprint beeper-design:LP_1 -> beeper-design:Pkg0201
- U15: renamed from C43; value 100n -> ~; footprint beeper-design:Pkg0201_39 -> beeper-design:LP_2
- U5: renamed from U2; footprint beeper-design:WLCSP_12 -> beeper-design:LP_4
- U9: renamed from C20; value 10n -> ~; footprint beeper-design:Pkg0201_30 -> beeper-design:LP_1
- moved U9 20.3 mm to (131.2, 109.1)
- moved R3 19.6 mm to (143.6, 100.8), turned to 90 degrees
- moved R7 17.0 mm to (145.3, 99.6), turned to 180 degrees
- moved R10 13.8 mm to (133.2, 109.8)
- moved R4 12.4 mm to (144.5, 100.1), turned to 90 degrees
- moved C23 11.2 mm to (148.3, 99.4), turned to 0 degrees
- moved R5 10.7 mm to (144.5, 102.1), turned to 270 degrees
- moved U15 8.69 mm to (137.8, 106.8)
- moved C4 8.51 mm to (145.6, 109.9)
- moved R15 7.46 mm to (133.1, 109.1), turned to 90 degrees
- moved U5 4.93 mm to (148.8, 113.7)
- moved ? 3.89 mm to (130.4, 115.8)
- moved ? 3.08 mm to (135.9, 115.4)
- moved C14 2.78 mm to (147.0, 103.3), turned to 180 degrees
- moved ? 1.71 mm to (134.3, 115.8)
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Connections:
- C14 pad 1: mcu_mcu-wpwr0_gpio -> GND
- C14 pad 2: GND -> VDD1P8
- C23 pad 1: VBUS -> GND
- C23 pad 2: D- -> RECT
- R10 pad 1: FOD -> board-io_qsen-i3c_scl
- R10 pad 2: GND -> mcu_q-spi_sck
- R15 pad 1: VDD1P8 -> board-io_qsen-i3c_scl
- R15 pad 2: mcu_dbg-m33_swdio -> VDD1P8
- R3 pad 1: RF2 -> FOD
- R3 pad 2: RF3 -> GND
- R4 pad 1: GND -> FOD
- R4 pad 2: V18P -> RECT
- R5 pad 1: mcu_hap-i2c_sda -> mcu_mcu-wpwr0_gpio
- R5 pad 2: VDD1P8 -> GND
- R7 pad 1: mcu_q-spi_sdi -> mcu_mcu-wpwr3_gpio
- R7 pad 2: TDMOUT -> GND
- U9 pad 1: AC2 -> mcu_q-spi_sdi
- U9 pad 2: BOOT2 -> TDMOUT
Routing:
- net GND: track 20.9 -> 25.7 mm, vias 49 -> 59
- net V18P: track 0.00 -> 3.88 mm
- net RECT: track 2.83 -> 5.68 mm
- net mcu_mcu-button2_gpio: track 10.8 -> 12.2 mm
- net mcu_mcu-wpwr3_gpio: track 19.6 -> 18.2 mm

Commit message: exported yet again
Parts:
- removed the C24 at (147.4, 99.4)
- removed the C7 at (139.3, 107.8)
- removed the D1 at (142.1, 103.0)
- removed the U12 at (133.2, 105.8)
- added C14: 2.2u, beeper-design:Pkg0201_25, F.Cu at (147.0, 103.3)
- added C2: 22u, beeper-design:Pkg0603, F.Cu at (143.5, 110.0)
- added C28: 1u, beeper-design:Pkg0201_5, F.Cu at (149.8, 106.9)
- added TP9: ~, beeper-design:SMD_TESTPT, B.Cu at (136.5, 107.4)
- C24: renamed from C9; value 10u -> 4.7u; footprint beeper-design:Pkg0402_7 -> beeper-design:Pkg0402_6
- C7: renamed from TP9; value ~ -> 10u; footprint beeper-design:SMD_TESTPT -> beeper-design:Pkg0402_1; moved to F.Cu
- C9: renamed from C28; value 1u -> 10u; footprint beeper-design:Pkg0201_5 -> beeper-design:Pkg0402_7
- D1: renamed from XTAL1; footprint beeper-design:CRYSTAL_SMD_4P_L2_0_W1_6_BL_1 -> beeper-design:LP_5
- U12: renamed from C14; value 2.2u -> ~; footprint beeper-design:Pkg0201_25 -> beeper-design:LP_8
- XTAL1: renamed from C2; value 22u -> ~; footprint beeper-design:Pkg0603 -> beeper-design:CRYSTAL_SMD_4P_L2_0_W1_6_BL_1
- moved U12 14.0 mm to (133.2, 105.8), turned to 90 degrees
- moved D1 12.3 mm to (142.1, 103.0), turned to 0 degrees
- moved C24 10.2 mm to (147.4, 99.4)
- moved C9 10.1 mm to (139.8, 106.2), turned to 0 degrees
- moved XTAL1 9.58 mm to (134.3, 112.5), turned to 270 degrees
- moved ? 5.57 mm to (130.4, 115.8)
- moved ? 3.95 mm to (135.9, 115.4)
- moved C7 2.76 mm to (139.3, 107.8), turned to 0 degrees
- moved ? 2.50 mm to (132.9, 115.8)
- moved ? 2.25 mm to (132.0, 116.0)
- moved ? 1.39 mm to (134.3, 115.8)
Connections:
- C24 pad 2: mcu_VBUS -> RECT
- C9 pad 2: VDD_MIC -> mcu_VBUS
- D1 pad 1: XTAL32Mp -> board-io_rgb_r
- D1 pad 2: GND -> VLED
- D1 pad 3: XTAL32Mm -> board-io_rgb_g
- D1 pad 4: GND -> board-io_rgb_b
- XTAL1 pad 1: GND -> XTAL32Mp
- XTAL1 pad 2: V14 -> GND

Commit message: exported yet again 2
Parts:
- removed the C24 at (147.4, 99.4)
- removed the C7 at (139.3, 107.8)
- removed the D1 at (142.1, 103.0)
- removed the U12 at (133.2, 105.8)
- added C14: 2.2u, beeper-design:Pkg0201_25, F.Cu at (147.0, 103.3)
- added C2: 22u, beeper-design:Pkg0603, F.Cu at (143.5, 110.0)
- added C28: 1u, beeper-design:Pkg0201_5, F.Cu at (149.8, 106.9)
- added TP9: ~, beeper-design:SMD_TESTPT, B.Cu at (136.5, 107.4)
- C24: renamed from C9; value 10u -> 4.7u; footprint beeper-design:Pkg0402_7 -> beeper-design:Pkg0402_6
- C7: renamed from TP9; value ~ -> 10u; footprint beeper-design:SMD_TESTPT -> beeper-design:Pkg0402_1; moved to F.Cu
- C9: renamed from C28; value 1u -> 10u; footprint beeper-design:Pkg0201_5 -> beeper-design:Pkg0402_7
- D1: renamed from XTAL1; footprint beeper-design:CRYSTAL_SMD_4P_L2_0_W1_6_BL_1 -> beeper-design:LP_5
- U12: renamed from C14; value 2.2u -> ~; footprint beeper-design:Pkg0201_25 -> beeper-design:LP_8
- XTAL1: renamed from C2; value 22u -> ~; footprint beeper-design:Pkg0603 -> beeper-design:CRYSTAL_SMD_4P_L2_0_W1_6_BL_1
- moved U12 14.0 mm to (133.2, 105.8), turned to 90 degrees
- moved D1 12.3 mm to (142.1, 103.0), turned to 0 degrees
- moved C24 10.2 mm to (147.4, 99.4)
- moved C9 10.1 mm to (139.8, 106.2), turned to 0 degrees
- moved XTAL1 9.58 mm to (134.3, 112.5), turned to 270 degrees
- moved ? 5.57 mm to (135.9, 115.4)
- moved ? 3.95 mm to (132.0, 116.0)
- moved C7 2.76 mm to (139.3, 107.8), turned to 0 degrees
- moved ? 2.50 mm to (130.4, 115.8)
- moved ? 2.25 mm to (134.3, 115.8)
- moved ? 1.39 mm to (132.9, 115.8)
Connections:
- C24 pad 2: mcu_VBUS -> RECT
- C9 pad 2: VDD_MIC -> mcu_VBUS
- D1 pad 1: XTAL32Mp -> board-io_rgb_r
- D1 pad 2: GND -> VLED
- D1 pad 3: XTAL32Mm -> board-io_rgb_g
- D1 pad 4: GND -> board-io_rgb_b
- XTAL1 pad 1: GND -> XTAL32Mp
- XTAL1 pad 2: V14 -> GND
Routing:
- net GND: track 25.7 -> 30.9 mm, vias 59 -> 63
