File: designs/beeper-design/kicad/beeper-design-2.kicad_sch (KiCad schematic)
At the start: 26 parts, among them U14 EVPBB4A9B000, U15 EVPBB4A9B000, U16 EVPBB4A9B000, U4 DA7212-01UM2, U9 LSM6DSOXTR

Commit message: another export
Parts:
- removed C26: 2.2u, beeper-design:Pkg0201_19, symbol C335106_10
- removed C27: 2.2u, beeper-design:Pkg0201_33, symbol C335106_21
- removed C28: 2.2u, beeper-design:Pkg0201_46, symbol C335106_28
- removed C29: 2.2u, beeper-design:Pkg0201_3, symbol C335106
- removed C30: 2.2u, beeper-design:Pkg0201_43, symbol C335106_27
- removed C31: 2.2u, beeper-design:Pkg0201, symbol C335106_36
- removed C32: 2.2u, beeper-design:Pkg0201_12, symbol C335106_6
- removed C37: 2.2u, beeper-design:Pkg0201_17, symbol C335106_8
- removed C38: 2.2u, beeper-design:Pkg0201_31, symbol C335106_20
- removed C39: 2.2u, beeper-design:Pkg0201_28, symbol C335106_18
- removed C42: 2.2u, beeper-design:Pkg0201_21, symbol C335106_11
- removed C43: 2.2u, beeper-design:Pkg0201_34, symbol C335106_22
- removed D1: HL-PCF-1617S39FU70GH203BC-A, beeper-design:LP_5, symbol C513368
- removed R10: 0R, beeper-design:Pkg0201_20, symbol my_resistor_5
- removed R12, R13: 8K2, beeper-design:Pkg0201_5, symbol my_resistor_1
- removed R14, R15: 8K2, beeper-design:Pkg0201_42, symbol my_resistor_10
- removed R9: 0R, beeper-design:Pkg0201_7, symbol my_resistor_2
- removed TP3, TP4: (no value), beeper-design:SMD_TESTPT, symbol smd_testpoint_cmp
- removed U14, U15, U16: EVPBB4A9B000, beeper-design:LP_2, symbol C140848
- removed U4: DA7212-01UM2, beeper-design:LP_3, symbol component
- removed U9: LSM6DSOXTR, beeper-design:LP_1, symbol LSM6DSOXTR
- added C1: 22u, beeper-design:Pkg0603, symbol C86295
- added C10: 2.2u, beeper-design:Pkg0201_18, symbol C335106_14
- added C11: 2.2u, beeper-design:Pkg0201_13, symbol C335106_11
- added C12: 2.2u, beeper-design:Pkg0201_31, symbol C335106_21
- added C2: 22u, beeper-design:Pkg0603_1, symbol C86295_1
- added C3: 22u, beeper-design:Pkg0603_2, symbol C86295_2
- added C36: 2.2u, beeper-design:Pkg0201_33, symbol C335106_23
- added C4: 47u, beeper-design:Pkg0805_1, symbol my_capacitor_1
- added C49: 2.2u, beeper-design:Pkg0201_44, symbol C335106_28
- added C5: 2.2u, beeper-design:Pkg0201_6, symbol C335106_4
- added C50: 2.2u, beeper-design:Pkg0201_8, symbol C335106_6
- added C6: 47u, beeper-design:Pkg0805, symbol my_capacitor
- added C7: 2.2u, beeper-design:Pkg0201_32, symbol C335106_22
- added C8: 2.2u, beeper-design:Pkg0201_46, symbol C335106_30
- added C9: 2.2u, beeper-design:Pkg0201_5, symbol C335106_3
- added J1: TC2030-IDC-NL, beeper-design:TC2030_IDC_NL_FOOTPRINT, symbol component
- added J6: 10103594-0001LF, beeper-design:AMPHENOL_10103594_0001LF, symbol AMPHENOL_10103594_0001LF
- added L1: 470n, beeper-design:Pkg0201_40, symbol my_inductor
- added L2: 470n, beeper-design:Pkg0201_54, symbol my_inductor_1
- added R1: 0R, beeper-design:Pkg0201_27, symbol my_resistor_6
- added R11: 0R, beeper-design:Pkg0201_53, symbol my_resistor_13
- added R18: 100K, beeper-design:Pkg0201_21, symbol my_resistor_4
- added R19: 0R, beeper-design:Pkg0201_19, symbol my_resistor_2
- added TP10, TP11, TP12, TP5, TP6, TP7, TP8, TP9: (no value), beeper-design:SMD_TESTPT, symbol smd_testpoint_cmp
- added U1: DA14705-00000HZ2, beeper-design:LP, symbol DA14705
- added U17: (no value), beeper-design:Pkg_2450AT18D0100_STD_R_1, symbol Sym2450AT18D0100001E
- added U7: TPD4S012DRYR, beeper-design:SON_6_L1_5_W1_0_P0_50_BL, symbol C96506
- added XTAL1: XRCGB32M000F1H00R0, beeper-design:CRYSTAL_SMD_4P_L2_0_W1_6_BL_1, symbol C880116
Connections:
- net GND: now also C1.1, C10.1, C11.1, C12.1, C2.1, C3.1, C36.2, C4.1, C49.2, C5.1, C50.2, C6.1, C7.1, C8.1, C9.1, J1.5, J6.5 (GND), R18.2, TP10.p, TP12.p, U1.A11 (RFIOM2), U1.A12 (PSUBRF), U1.A8 (PSUB), U1.A9 (RFIOM1), U1.B9 (ESDN), U1.C12 (GND_RF2), U1.C2 (VSSIOQQ), U1.D12 (GND_RF1), U1.E11 (GND_XTAL2), U1.E12 (GND_XTAL1), U1.F5 (VSSD4), U1.F6 (VSSD3), U1.G12 (GND_XTAL3), U1.G5 (VSSD1), U1.G6 (VSSD2), U1.G7 (VSSD5), U1.H1 (GND_BOOST), U1.H6 (AVS1), U1.H7 (AVS2), U1.H8 (AVS3), U1.L8 (GND_SDADC), U1.L9 (GND_VAD), U1.M1 (GND_BUCK), U17.2 (GND), U17.3 (GND), U17.4 (GND), U7.4 (GND), XTAL1.2 (GND1), XTAL1.4 (GND0)
- net VDD1P8: now also C4.2, U1.K2 (V18)
- net VLED: now also C10.2, U1.K1 (VLED)
- net board-io_qsen-i3c_scl: now also U1.K9 (P1_12)
- net board-io_rgb_b: now also U1.L4 (LED3)
- net board-io_rgb_g: now also U1.L6 (LED2)
- net board-io_rgb_r: now also U1.L5 (LED1)
- net codec-i2c-net_scl: now also U1.B1 (P2_04)
- net codec-i2c-net_sda: now also U1.H2 (P0_22)
- net mcu_mcu-button0_gpio: now also U1.D11 (P0_28)
- net mcu_mcu-button1_gpio: now also U1.M8 (P1_06)
- net mcu_mcu-button2_gpio: now also U1.H3 (P1_26)
- net mcu_q-spi_cs: now also U1.H11 (P2_09)
- net mcu_q-spi_sck: now also U1.H12 (P2_08)
- net mcu_q-spi_sdi: now also U1.H10 (P0_30)
- net mcu_q-spi_sdo: now also U1.L7 (P0_27)
- new net: C8.2, TP11.p, U1.M4 (VBAT)
- new net: C2.2, C3.2, U1.A7 (V14RF), U1.L2 (V14)
- new net: L1.1, U1.M2 (LX)
- new net: L1.2, U1.L1 (LY)
- new net: TP9.p, U1.K6 (P1_23)
- new net: TP7.p, U1.K7 (P1_22)
- new net: TP8.p, U1.J7 (P1_31)
- new net: C1.2, U1.L3 (V12)
- new net: J1.2, U1.C7 (P0_00)
- new net: J1.3, U1.G8 (P0_16)
- new net: J1.4, U1.D6 (P0_01)
- new net: J1.6, U1.G9 (P0_10)
- new net: U1.F11 (XTAL32Mp), XTAL1.1
- new net: U1.F12 (XTAL32Mm), XTAL1.3
- new net: U1.J10 (NC), U1.J11 (NC), U1.J12 (NC), U1.K10 (NC), U1.K11 (NC), U1.K12 (NC), U1.L10 (NC), U1.L11 (NC), U1.L12 (NC), U1.M10 (NC), U1.M11 (NC), U1.M12 (NC)
- new net: TP5.p, U1.K5 (P0_31)
- new net: TP6.p, U1.J8 (P1_30)
- new net: L2.1, U1.J1 (LZ)
- new net D+: J6.3 (D+), U1.F1 (P2_10), U7.1 (D+)
- new net D-: J6.2 (D-), U1.G1 (P2_11), U7.2 (D-)
- new net RF1: C49.1, R11.1, U1.A10 (RFIOP)
- new net RF2: C50.1, R11.2, R19.1
- new net RF3: R19.2, U17.1 (ANT)
- new net SHIELD: C36.1, J6.10 (SHIELD), J6.11 (SHIELD), J6.13 (SHIELD), J6.14 (SHIELD), J6.6 (SHIELD), J6.7 (SHIELD), J6.8 (SHIELD), J6.9 (SHIELD), R18.1
- new net V18F: C5.2, R1.1, U1.C1 (V18F)
- new net VBUS: C9.2, J1.1, J6.1 (VCC), U1.M5 (VBUS), U7.6 (VBUS)
- new net VDD1P8P: C6.2, R1.2, U1.J2 (V18P)
- new net VDD3P0: C7.2, U1.M6 (V30)
- new net VDDSYS: C11.2, C12.2, L2.2, U1.M3 (VSYS)
- new net board-io_qsen-i3c_sda: U1.K8 (P1_11)
- new net mcu_hap-gpio0_gpio: U1.J9 (P2_01)
- new net mcu_hap-gpio1_gpio: U1.H9 (P0_23)
- new net mcu_hap-i2c_scl: U1.G10 (P0_08)
- new net mcu_hap-i2c_sda: U1.M7 (P1_05)
- new net mcu_mcu-mem_cs: U1.J3 (P1_24)
- new net mcu_mcu-mem_sck: U1.F4 (P1_19)
- new net mcu_mcu-mem_sdio0: U1.J6 (P1_15)
- new net mcu_mcu-mem_sdio1: U1.G2 (P1_14)
- new net mcu_mcu-mem_sdio2: U1.H4 (P1_13)
- new net mcu_mcu-mem_sdio3: U1.F3 (P1_20)
- new net mcu_mcu-wpwr0_gpio: U1.K4 (P1_00)
- new net mcu_mcu-wpwr1_gpio: U1.J4 (P1_09)
- new net mcu_mcu-wpwr2_gpio: U1.K3 (P1_07)
- new net mcu_mcu-wpwr3_gpio: U1.J5 (P1_25)
- no-connect marks 7 -> 1

Commit message: new export
Parts:
- removed C10: 2.2u, beeper-design:Pkg0201_18, symbol C335106_14
- removed C11: 2.2u, beeper-design:Pkg0201_13, symbol C335106_11
- removed C12: 2.2u, beeper-design:Pkg0201_31, symbol C335106_21
- removed C36: 2.2u, beeper-design:Pkg0201_33, symbol C335106_23
- removed C49: 2.2u, beeper-design:Pkg0201_44, symbol C335106_28
- removed C5: 2.2u, beeper-design:Pkg0201_6, symbol C335106_4
- removed C50: 2.2u, beeper-design:Pkg0201_8, symbol C335106_6
- removed C7: 2.2u, beeper-design:Pkg0201_32, symbol C335106_22
- removed C8: 2.2u, beeper-design:Pkg0201_46, symbol C335106_30
- removed C9: 2.2u, beeper-design:Pkg0201_5, symbol C335106_3
- removed J6: 10103594-0001LF, beeper-design:AMPHENOL_10103594_0001LF, symbol AMPHENOL_10103594_0001LF
- removed R1: 0R, beeper-design:Pkg0201_27, symbol my_resistor_6
- removed R19: 0R, beeper-design:Pkg0201_19, symbol my_resistor_2
- added C10: 2.2u, beeper-design:Pkg0201_12, symbol C335106_9
- added C11: 2.2u, beeper-design:Pkg0201_5, symbol C335106_3
- added C12: 2.2u, beeper-design:Pkg0201_25, symbol C335106_16
- added C36: 2.2u, beeper-design:Pkg0201_30, symbol C335106_19
- added C49: 2.2u, beeper-design:Pkg0201_37, symbol C335106_23
- added C5: 2.2u, beeper-design:Pkg0201_1, symbol C335106_36
- added C50: 2.2u, beeper-design:Pkg0201_2, symbol C335106
- added C7: 2.2u, beeper-design:Pkg0201_26, symbol C335106_17
- added C8: 2.2u, beeper-design:Pkg0201_41, symbol C335106_25
- added C9: 2.2u, beeper-design:Pkg0201_54, symbol C335106_34
- added J6: (no value), beeper-design:GCT_USB3100_XX_X_REVB_1, symbol component_1
- added R1: 0R, beeper-design:Pkg0201_19, symbol my_resistor_5
- added R19: 0R, beeper-design:Pkg0201_13, symbol my_resistor_1
- L1: footprint beeper-design:Pkg0201_40 -> beeper-design:Pkg0201_32
- L2: footprint beeper-design:Pkg0201_54 -> beeper-design:Pkg0201_46
- R11: footprint beeper-design:Pkg0201_53 -> beeper-design:Pkg0201_45
- R18: footprint beeper-design:Pkg0201_21 -> beeper-design:Pkg0201_17
Connections:
- net D+: now also J6.3 (D+)
- net D-: now also J6.2 (D-)
- net GND: now also C10.1, C11.1, C12.1, C36.2, C49.2, C5.1, C50.2, C7.1, C8.1, C9.1, J6.5 (GND)
- net RF1: now also C49.1
- net RF2: now also C50.1, R19.1
- net RF3: now also R19.2
- net SHIELD: now also C36.1, J6.6 (SHIELD), J6.7 (SHIELD), J6.8 (SHIELD), J6.9 (SHIELD)
- net V18F: now also C5.2, R1.1
- net VBUS: now also C9.2, J6.1 (VBUS)
- net VDD1P8P: now also R1.2
- net VDD3P0: now also C7.2
- net VDDSYS: now also C11.2, C12.2
- net VLED: now also C10.2
- net at TP11.p, U1.M4 (VBAT): now also C8.2

Commit message: exported, yet XTALM32p keeps disappearing
Parts:
- removed C10: 2.2u, beeper-design:Pkg0201_12, symbol C335106_9
- removed C11: 2.2u, beeper-design:Pkg0201_5, symbol C335106_3
- removed C12: 2.2u, beeper-design:Pkg0201_25, symbol C335106_16
- removed C36: 2.2u, beeper-design:Pkg0201_30, symbol C335106_19
- removed C4: 47u, beeper-design:Pkg0805_1, symbol my_capacitor_1
- removed C49: 2.2u, beeper-design:Pkg0201_37, symbol C335106_23
- removed C5: 2.2u, beeper-design:Pkg0201_1, symbol C335106_36
- removed C50: 2.2u, beeper-design:Pkg0201_2, symbol C335106
- removed C7: 2.2u, beeper-design:Pkg0201_26, symbol C335106_17
- removed C8: 2.2u, beeper-design:Pkg0201_41, symbol C335106_25
- removed C9: 2.2u, beeper-design:Pkg0201_54, symbol C335106_34
- removed L2: 470n, beeper-design:Pkg0201_46, symbol my_inductor_1
- removed R1: 0R, beeper-design:Pkg0201_19, symbol my_resistor_5
- removed R11: 0R, beeper-design:Pkg0201_45, symbol my_resistor_13
- removed R18: 100K, beeper-design:Pkg0201_17, symbol my_resistor_4
- removed R19: 0R, beeper-design:Pkg0201_13, symbol my_resistor_1
- added C10: 2.2u, beeper-design:Pkg0201_27, symbol C335106_1
- added C11: 10u, beeper-design:Pkg0402_6, symbol C105225_5
- added C12: 10u, beeper-design:Pkg0402_5, symbol C105225_4
- added C13: 1u, beeper-design:Pkg0201_29, symbol my_capacitor_15
- added C36: 100n, beeper-design:Pkg0201_7, symbol my_capacitor_5
- added C4: 47u, beeper-design:Pkg0805_1, symbol my_capacitor_19
- added C49: 1p, beeper-design:Pkg0201_5, symbol my_capacitor_3
- added C5: 100n, beeper-design:Pkg0201_39, symbol my_capacitor_23
- added C50: 1p, beeper-design:Pkg0201_15, symbol my_capacitor_8
- added C7: 10u, beeper-design:Pkg0402, symbol C105225
- added C8: 10u, beeper-design:Pkg0402_1, symbol C105225_1
- added C9: 10u, beeper-design:Pkg0402_2, symbol C105225_2
- added L2: 1u, beeper-design:Pkg0402_3, symbol C531288
- added R1: 0R, beeper-design:Pkg0201_14, symbol my_resistor_7
- added R11: 0R, beeper-design:Pkg0201_10, symbol my_resistor_5
- added R12, R13: 8K2, beeper-design:Pkg0201_28, symbol my_resistor_11
- added R14, R15: 8K2, beeper-design:Pkg0201_42, symbol my_resistor_14
- added R18: 100K, beeper-design:Pkg0201_47, symbol my_resistor_16
- added R19: 0R, beeper-design:Pkg0201_19, symbol my_resistor_9
- added U2: AT25FF321A-UUN-T, beeper-design:WLCSP_12, symbol AT25FF321A_UUN_T
- added U5: FH19C-6S-0.5SH(10), beeper-design:LP_4, symbol FH19C_6S_0_5SH_10_
- J1, J6, TP10, TP11, TP12, TP5, TP6, TP7, TP8, TP9, U7: now fitted; now in the parts list
- L1: footprint beeper-design:Pkg0201_32 -> beeper-design:Pkg0201_21
Connections:
- net D+: now also U1.F1 (P2_10); no longer U1.F1 (P2_10)
- net D-: now also U1.G1 (P2_11); no longer U1.G1 (P2_11)
- net GND: now also U1.A11 (RFIOM2), U1.A12 (PSUBRF), U1.A8 (PSUB), U1.A9 (RFIOM1), U1.B9 (ESDN), U1.C12 (GND_RF2), U1.C2 (VSSIOQQ), U1.D12 (GND_RF1), U1.E11 (GND_XTAL2), U1.E12 (GND_XTAL1), U1.F5 (VSSD4), U1.F6 (VSSD3), U1.G12 (GND_XTAL3), U1.G5 (VSSD1), U1.G6 (VSSD2), U1.G7 (VSSD5), U1.H1 (GND_BOOST), U1.H6 (AVS1), U1.H7 (AVS2), U1.H8 (AVS3), U1.L8 (GND_SDADC), U1.L9 (GND_VAD), U1.M1 (GND_BUCK), C10.1, C11.1, C12.1, C13.1, C36.2, C4.1, C49.2, C5.1, C50.2, C7.1, C8.1, C9.1, R18.2, U2.C3 (GND), U5.2, U5.3, U5.4, U5.7, U5.8; no longer U1.A11 (RFIOM2), U1.A12 (PSUBRF), U1.A8 (PSUB), U1.A9 (RFIOM1), U1.B9 (ESDN), U1.C12 (GND_RF2), U1.C2 (VSSIOQQ), U1.D12 (GND_RF1), U1.E11 (GND_XTAL2), U1.E12 (GND_XTAL1), U1.F5 (VSSD4), U1.F6 (VSSD3), U1.G12 (GND_XTAL3), U1.G5 (VSSD1), U1.G6 (VSSD2), U1.G7 (VSSD5), U1.H1 (GND_BOOST), U1.H6 (AVS1), U1.H7 (AVS2), U1.H8 (AVS3), U1.L8 (GND_SDADC), U1.L9 (GND_VAD), U1.M1 (GND_BUCK)
- net RF1: now also U1.A10 (RFIOP), C49.1, R11.1; no longer U1.A10 (RFIOP)
- net RF2: now also C50.1, R11.2, R19.1
- net RF3: now also R19.2
- net SHIELD: now also C36.1, R18.1
- net V18F: now also U1.C1 (V18F), C13.2, C5.2, R1.1, U2.B2 (Vcc); no longer U1.C1 (V18F)
- net VBUS: now also U1.M5 (VBUS), C9.2; no longer U1.M5 (VBUS)
- net VDD1P8: now also U1.K2 (V18), C4.2, R14.2, R15.2; no longer U1.K2 (V18)
- net VDD1P8P: now also U1.J2 (V18P), R1.2, R12.2, R13.2; no longer U1.J2 (V18P)
- net VDD3P0: now also U1.M6 (V30), C7.2; no longer U1.M6 (V30)
- net VDDSYS: now also U1.M3 (VSYS), C11.2, C12.2, L2.2; no longer U1.M3 (VSYS)
- net VLED: now also U1.K1 (VLED), C10.2; no longer U1.K1 (VLED)
- net at XTAL1.1: now also U1.F11 (XTAL32Mp); no longer U1.F11 (XTAL32Mp)
- net at XTAL1.3: now also U1.F12 (XTAL32Mm); no longer U1.F12 (XTAL32Mm)
- net mcu_data2: now reaches TP8.p
- net mcu_data2: now also U1.J7 (P1_31); no longer U1.J7 (P1_31)
- net at C2.2, C3.2: now also U1.A7 (V14RF), U1.L2 (V14); no longer U1.A7 (V14RF), U1.L2 (V14)
- net at L1.2: now also U1.L1 (LY); no longer U1.L1 (LY)
- net at C1.2: now also U1.L3 (V12); no longer U1.L3 (V12)
- net at L1.1: now also U1.M2 (LX); no longer U1.M2 (LX)
- net at TP11.p: now also U1.M4 (VBAT), C8.2; no longer U1.M4 (VBAT)
- net mcu_data3: now reaches TP9.p
- net mcu_data3: now also U1.K6 (P1_23); no longer U1.K6 (P1_23)
- net mcu_clk: now reaches TP5.p
- net mcu_clk: now also U1.K5 (P0_31); no longer U1.K5 (P0_31)
- net mcu_data1: now reaches TP7.p
- net mcu_data1: now also U1.K7 (P1_22); no longer U1.K7 (P1_22)
- net mcu_data0: now reaches TP6.p
- net mcu_data0: now also U1.J8 (P1_30); no longer U1.J8 (P1_30)
- net mcu_swdio: now reaches J1.2
- net mcu_swdio: now also U1.C7 (P0_00); no longer U1.C7 (P0_00)
- net mcu_rx: now reaches J1.3
- net mcu_rx: now also U1.H10 (P0_30); no longer U1.G8 (P0_16)
- net mcu_swdclk: now reaches J1.4
- net mcu_swdclk: now also U1.D6 (P0_01); no longer U1.D6 (P0_01)
- net mcu_tx: now reaches J1.6
- net mcu_tx: now also U1.B11 (P0_18); no longer U1.G9 (P0_10)
- removed net board-io_qsen-i3c_scl: U1.K9 (P1_12)
- removed net board-io_qsen-i3c_sda: U1.K8 (P1_11)
- removed net board-io_rgb_b: U1.L4 (LED3)
- removed net board-io_rgb_g: U1.L6 (LED2)
- removed net board-io_rgb_r: U1.L5 (LED1)
- removed net codec-i2c-net_scl: U1.B1 (P2_04)
- removed net codec-i2c-net_sda: U1.H2 (P0_22)
- removed net mcu_hap-gpio0_gpio: U1.J9 (P2_01)
- removed net mcu_hap-gpio1_gpio: U1.H9 (P0_23)
- removed net mcu_hap-i2c_scl: U1.G10 (P0_08)
- removed net mcu_hap-i2c_sda: U1.M7 (P1_05)
- removed net mcu_mcu-button0_gpio: U1.D11 (P0_28)
- removed net mcu_mcu-button1_gpio: U1.M8 (P1_06)
- removed net mcu_mcu-button2_gpio: U1.H3 (P1_26)
- removed net mcu_mcu-mem_cs: U1.J3 (P1_24)
- removed net mcu_mcu-mem_sck: U1.F4 (P1_19)
- removed net mcu_mcu-mem_sdio0: U1.J6 (P1_15)
- removed net mcu_mcu-mem_sdio1: U1.G2 (P1_14)
- removed net mcu_mcu-mem_sdio2: U1.H4 (P1_13)
- removed net mcu_mcu-mem_sdio3: U1.F3 (P1_20)
- removed net mcu_mcu-wpwr0_gpio: U1.K4 (P1_00)
- removed net mcu_mcu-wpwr1_gpio: U1.J4 (P1_09)
- removed net mcu_mcu-wpwr2_gpio: U1.K3 (P1_07)
- removed net mcu_mcu-wpwr3_gpio: U1.J5 (P1_25)
- removed net mcu_q-spi_cs: U1.H11 (P2_09)
- removed net mcu_q-spi_sck: U1.H12 (P2_08)
- removed net mcu_q-spi_sdi: U1.H10 (P0_30)
- removed net mcu_q-spi_sdo: U1.L7 (P0_27)
- new net: L2.1, U1.J1 (LZ)
- new net: U1.J10 (NC), U1.J11 (NC), U1.J12 (NC), U1.K10 (NC), U1.K11 (NC), U1.K12 (NC), U1.L10 (NC), U1.L11 (NC), U1.L12 (NC), U1.M10 (NC), U1.M11 (NC), U1.M12 (NC)
- new net: U2.A1 (NC), U2.A5 (NC), U2.G1 (NC), U2.G5 (NC)
- new net MICBIAS1: U5.6
- new net board-io_b: U1.L4 (LED3)
- new net board-io_clk: U5.1
- new net board-io_data: U5.5
- new net board-io_g: U1.L6 (LED2)
- new net board-io_r: U1.L5 (LED1)
- new net mcu0_gpio: U1.D11 (P0_28)
- new net mcu0_gpio1: U1.C10 (P0_11)
- new net mcu0_gpio2: U1.E3 (P2_00)
- new net mcu1_gpio: U1.E9 (P0_14)
- new net mcu1_gpio1: U1.M8 (P1_06)
- new net mcu1_gpio2: U1.E1 (P0_13)
- new net mcu2_gpio: U1.D2 (P2_12)
- new net mcu2_gpio1: U1.C4 (P0_26)
- new net mcu3_gpio: U1.F2 (P1_28)
- new net mcu_cs: U1.H9 (P0_23)
- new net mcu_cs1: U1.A6 (OQSIF_CS), U2.B4 (CSn)
- new net mcu_sck: U1.J9 (P2_01)
- new net mcu_sck1: U1.B4 (OQSIF_CLK), U2.F2 (SCK)
- new net mcu_scl: R15.1, U1.K9 (P1_12)
- new net mcu_scl1: U1.E10 (P0_21)
- new net mcu_scl2: R13.1, U1.C3 (P0_25)
- new net mcu_sda: R12.1, U1.D4 (P0_12)
- new net mcu_sda1: U1.C11 (P0_29)
- new net mcu_sda2: R14.1, U1.K8 (P1_11)
- new net mcu_sdi: U1.M7 (P1_05)
- new net mcu_sdio0: U1.A1 (OQSIF_D0), U2.E3 (SI)
- new net mcu_sdio1: U1.A2 (OQSIF_D1), U2.D4 (SO)
- new net mcu_sdio2: U1.A3 (OQSIF_D2), U2.F4 (WPn)
- new net mcu_sdio3: U1.B3 (OQSIF_D3), U2.D2 (HRn)
- new net mcu_sdo: U1.L7 (P0_27)
- no-connect marks 1 -> 3

Commit message: fixed up pours, keepout regions
Parts:
- removed C13: 1u, beeper-design:Pkg0201_29, symbol my_capacitor_15
- removed C36: 100n, beeper-design:Pkg0201_7, symbol my_capacitor_5
- removed C4: 47u, beeper-design:Pkg0805_1, symbol my_capacitor_19
- removed C49: 1p, beeper-design:Pkg0201_5, symbol my_capacitor_3
- removed C5: 100n, beeper-design:Pkg0201_39, symbol my_capacitor_23
- removed C50: 1p, beeper-design:Pkg0201_15, symbol my_capacitor_8
- removed C6: 47u, beeper-design:Pkg0805, symbol my_capacitor
- removed R1: 0R, beeper-design:Pkg0201_14, symbol my_resistor_7
- removed R11: 0R, beeper-design:Pkg0201_10, symbol my_resistor_5
- removed R12, R13: 8K2, beeper-design:Pkg0201_28, symbol my_resistor_11
- removed R14, R15: 8K2, beeper-design:Pkg0201_42, symbol my_resistor_14
- removed R18: 100K, beeper-design:Pkg0201_47, symbol my_resistor_16
- removed R19: 0R, beeper-design:Pkg0201_19, symbol my_resistor_9
- added C13: 1u, beeper-design:Pkg0201_43, symbol my_capacitor_21
- added C36: 100n, beeper-design:Pkg0201_21, symbol my_capacitor_11
- added C4: 47u, beeper-design:Pkg0805_1, symbol my_capacitor_25
- added C49: 1p, beeper-design:Pkg0201_19, symbol my_capacitor_9
- added C5: 100n, beeper-design:Pkg0201_5, symbol my_capacitor_2
- added C50: 1p, beeper-design:Pkg0201_29, symbol my_capacitor_14
- added C6: 47u, beeper-design:Pkg0805, symbol my_capacitor_6
- added R1: 0R, beeper-design:Pkg0201_28, symbol my_resistor_12
- added R11: 0R, beeper-design:Pkg0201_24, symbol my_resistor_10
- added R12, R13: 8K2, beeper-design:Pkg0201_42, symbol my_resistor_16
- added R14, R15: 8K2, beeper-design:Pkg0201_8, symbol my_resistor_2
- added R18: 100K, beeper-design:Pkg0201_13, symbol my_resistor_4
- added R19: 0R, beeper-design:Pkg0201_33, symbol my_resistor_14
- C10: footprint beeper-design:Pkg0201_27 -> beeper-design:Pkg0201_41
- C11: footprint beeper-design:Pkg0402_6 -> beeper-design:Pkg0402_8
- C12: footprint beeper-design:Pkg0402_5 -> beeper-design:Pkg0402_7
- C7: footprint beeper-design:Pkg0402 -> beeper-design:Pkg0402_2
- C8: footprint beeper-design:Pkg0402_1 -> beeper-design:Pkg0402_3
- C9: footprint beeper-design:Pkg0402_2 -> beeper-design:Pkg0402_4
- L1: footprint beeper-design:Pkg0201_21 -> beeper-design:Pkg0201_35
- L2: footprint beeper-design:Pkg0402_3 -> beeper-design:Pkg0402_5
- U1: footprint beeper-design:LP -> beeper-design:LP_3
- U5: footprint beeper-design:LP_4 -> beeper-design:LP_7
Connections:
- net GND: now also C13.1, C36.2, C4.1, C49.2, C5.1, C50.2, C6.1, R18.2
- net RF1: now also C49.1, R11.1
- net RF2: now also C50.1, R11.2, R19.1
- net RF3: now also R19.2
- net SHIELD: now also C36.1, R18.1
- net V18F: now also C13.2, C5.2, R1.1
- net VDD1P8: now also C4.2, R14.2, R15.2
- net VDD1P8P: now also C6.2, R1.2, R12.2, R13.2
- net mcu_scl: now also R15.1
- net mcu_scl2: now also R13.1
- net mcu_sda: now also R12.1
- net mcu_sda2: now also R14.1

Commit message: exported to Kicad, fixed Kicad, exported gerbers
Parts:
- removed C1: 22u, beeper-design:Pkg0603, symbol C86295
- removed C10: 2.2u, beeper-design:Pkg0201_41, symbol C335106_1
- removed C11: 10u, beeper-design:Pkg0402_8, symbol C105225_5
- removed C12: 10u, beeper-design:Pkg0402_7, symbol C105225_4
- removed C13: 1u, beeper-design:Pkg0201_43, symbol my_capacitor_21
- removed C2: 22u, beeper-design:Pkg0603_1, symbol C86295_1
- removed C3: 22u, beeper-design:Pkg0603_2, symbol C86295_2
- removed C36: 100n, beeper-design:Pkg0201_21, symbol my_capacitor_11
- removed C4: 47u, beeper-design:Pkg0805_1, symbol my_capacitor_25
- removed C49: 1p, beeper-design:Pkg0201_19, symbol my_capacitor_9
- removed C5: 100n, beeper-design:Pkg0201_5, symbol my_capacitor_2
- removed C50: 1p, beeper-design:Pkg0201_29, symbol my_capacitor_14
- removed C6: 47u, beeper-design:Pkg0805, symbol my_capacitor_6
- removed C7: 10u, beeper-design:Pkg0402_2, symbol C105225
- removed C8: 10u, beeper-design:Pkg0402_3, symbol C105225_1
- removed C9: 10u, beeper-design:Pkg0402_4, symbol C105225_2
- removed J1: TC2030-IDC-NL, beeper-design:TC2030_IDC_NL_FOOTPRINT, symbol component
- removed J6: (no value), beeper-design:GCT_USB3100_XX_X_REVB_1, symbol component_1
- removed R1: 0R, beeper-design:Pkg0201_28, symbol my_resistor_12
- removed R11: 0R, beeper-design:Pkg0201_24, symbol my_resistor_10
- removed R12, R13: 8K2, beeper-design:Pkg0201_42, symbol my_resistor_16
- removed R14, R15: 8K2, beeper-design:Pkg0201_8, symbol my_resistor_2
- removed R18: 100K, beeper-design:Pkg0201_13, symbol my_resistor_4
- removed R19: 0R, beeper-design:Pkg0201_33, symbol my_resistor_14
- added C1: 22u, beeper-design:Pkg0603_2, symbol C86295_2
- added C10: 2.2u, beeper-design:Pkg0201_8, symbol C335106
- added C11: 10u, beeper-design:Pkg0402_4, symbol C105225_3
- added C12: 10u, beeper-design:Pkg0402_3, symbol C105225_2
- added C13: 1u, beeper-design:Pkg0201_10, symbol my_capacitor_4
- added C2: 22u, beeper-design:Pkg0603, symbol C86295
- added C3: 22u, beeper-design:Pkg0603_1, symbol C86295_1
- added C36: 100n, beeper-design:Pkg0201_36, symbol my_capacitor_21
- added C4: 47u, beeper-design:Pkg0805, symbol my_capacitor_8
- added C49: 1p, beeper-design:Pkg0201_34, symbol my_capacitor_19
- added C5: 100n, beeper-design:Pkg0201_20, symbol my_capacitor_12
- added C50: 1p, beeper-design:Pkg0201_44, symbol my_capacitor_24
- added C6: 47u, beeper-design:Pkg0805_1, symbol my_capacitor_16
- added C7: 10u, beeper-design:Pkg0402_7, symbol C105225_4
- added C8: 10u, beeper-design:Pkg0402_8, symbol C105225_5
- added C9: 10u, beeper-design:Pkg0402, symbol C105225
- added J1: TC2030-IDC-NL, beeper-design:TC2030_IDC_NL_FOOTPRINT, symbol component_1
- added J6: (no value), beeper-design:GCT_USB3100_XX_X_REVB_1, symbol component_2
- added R1: 0R, beeper-design:Pkg0201_43, symbol my_resistor_14
- added R11: 0R, beeper-design:Pkg0201_39, symbol my_resistor_12
- added R12, R13: 8K2, beeper-design:Pkg0201_9, symbol my_resistor_1
- added R14, R15: 8K2, beeper-design:Pkg0201_23, symbol my_resistor_4
- added R18: 100K, beeper-design:Pkg0201_28, symbol my_resistor_6
- added R19: 0R, beeper-design:Pkg0201, symbol my_resistor_16
- L1: footprint beeper-design:Pkg0201_35 -> beeper-design:Pkg0201_2
- L2: footprint beeper-design:Pkg0402_5 -> beeper-design:Pkg0402_1
- U1: footprint beeper-design:LP_3 -> beeper-design:LP
- U5: footprint beeper-design:LP_7 -> beeper-design:LP_4
Connections:
- net D+: now also J6.3 (D+)
- net D-: now also J6.2 (D-)
- net GND: now also C1.1, C10.1, C11.1, C12.1, C13.1, C2.1, C3.1, C36.2, C4.1, C49.2, C5.1, C50.2, C6.1, C7.1, C8.1, C9.1, J1.5, J6.5 (GND), R18.2
- net RF1: now also C49.1, R11.1
- net RF2: now also C50.1, R11.2, R19.1
- net RF3: now also R19.2
- net SHIELD: now also C36.1, J6.6 (SHIELD), J6.7 (SHIELD), J6.8 (SHIELD), J6.9 (SHIELD), R18.1
- net V18F: now also C13.2, C5.2, R1.1
- net VBUS: now also C9.2, J1.1, J6.1 (VBUS)
- net VDD1P8: now also C4.2, R14.2, R15.2
- net VDD1P8P: now also C6.2, R1.2, R12.2, R13.2
- net VDD3P0: now also C7.2
- net VDDSYS: now also C11.2, C12.2
- net VLED: now also C10.2
- net mcu_rx: now also J1.3
- net mcu_scl: now also R15.1
- net mcu_scl2: now also R13.1
- net mcu_sda: now also R12.1
- net mcu_sda2: now also R14.1
- net mcu_swdclk: now also J1.4
- net mcu_swdio: now also J1.2
- net mcu_tx: now also J1.6
- net at U1.A7 (V14RF), U1.L2 (V14): now also C2.2, C3.2
- net at U1.L3 (V12): now also C1.2
- net at TP11.p, U1.M4 (VBAT): now also C8.2
