File: designs/beeper-design/kicad/beeper-design-2.kicad_sch (KiCad schematic)
At the start: 42 parts, among them J1 TC2030-IDC-NL, U1 DA14705-00000HZ2, U2 AT25FF321A-UUN-T, U5 FH19C-6S-0.5SH(10), U7 TPD4S012DRYR

Commit message: latest fully routed version
Parts:
- removed C1: 22u, beeper-design:Pkg0603_2, symbol C86295_2
- removed C11: 10u, beeper-design:Pkg0402_4, symbol C105225_3
- removed C12: 10u, beeper-design:Pkg0402_3, symbol C105225_2
- removed C13: 1u, beeper-design:Pkg0201_10, symbol my_capacitor_4
- removed C2: 22u, beeper-design:Pkg0603, symbol C86295
- removed C3: 22u, beeper-design:Pkg0603_1, symbol C86295_1
- removed C36: 100n, beeper-design:Pkg0201_36, symbol my_capacitor_21
- removed C4: 47u, beeper-design:Pkg0805, symbol my_capacitor_8
- removed C49: 1p, beeper-design:Pkg0201_34, symbol my_capacitor_19
- removed C5: 100n, beeper-design:Pkg0201_20, symbol my_capacitor_12
- removed C50: 1p, beeper-design:Pkg0201_44, symbol my_capacitor_24
- removed C6: 47u, beeper-design:Pkg0805_1, symbol my_capacitor_16
- removed C7: 10u, beeper-design:Pkg0402_7, symbol C105225_4
- removed C8: 10u, beeper-design:Pkg0402_8, symbol C105225_5
- removed C9: 10u, beeper-design:Pkg0402, symbol C105225
- removed J6: (no value), beeper-design:GCT_USB3100_XX_X_REVB_1, symbol component_2
- removed R1: 0R, beeper-design:Pkg0201_43, symbol my_resistor_14
- removed R11: 0R, beeper-design:Pkg0201_39, symbol my_resistor_12
- removed R12, R13: 8K2, beeper-design:Pkg0201_9, symbol my_resistor_1
- removed R14, R15: 8K2, beeper-design:Pkg0201_23, symbol my_resistor_4
- removed R18: 100K, beeper-design:Pkg0201_28, symbol my_resistor_6
- removed R19: 0R, beeper-design:Pkg0201, symbol my_resistor_16
- removed U2: AT25FF321A-UUN-T, beeper-design:WLCSP_12, symbol AT25FF321A_UUN_T
- removed U5: FH19C-6S-0.5SH(10), beeper-design:LP_4, symbol FH19C_6S_0_5SH_10_
- added C1: 22u, beeper-design:Pkg0603_1, symbol C86295_1
- added C11: 10u, beeper-design:Pkg0402_7, symbol C105225_4
- added C12: 10u, beeper-design:Pkg0402, symbol C105225
- added C2: 22u, beeper-design:Pkg0603_2, symbol C86295_2
- added C3: 22u, beeper-design:Pkg0603, symbol C86295
- added C4: 47u, beeper-design:Pkg0805, symbol my_capacitor_10
- added C49: 1p, beeper-design:Pkg0201_13, symbol my_capacitor_7
- added C5: 100n, beeper-design:Pkg0201_29, symbol my_capacitor_17
- added C50: 1p, beeper-design:Pkg0201_32, symbol my_capacitor_18
- added C6: 47u, beeper-design:Pkg0805_1, symbol my_capacitor_22
- added C7: 10u, beeper-design:Pkg0402_2, symbol C105225_1
- added C8: 10u, beeper-design:Pkg0402_4, symbol C105225_2
- added C9: 10u, beeper-design:Pkg0402_6, symbol C105225_3
- added R1: 0R, beeper-design:Pkg0201_47, symbol my_resistor_16
- added R11: 0R, beeper-design:Pkg0201_22, symbol my_resistor_8
- added R19: 0R, beeper-design:Pkg0201_39, symbol my_resistor_13
- C10: footprint beeper-design:Pkg0201_8 -> beeper-design:Pkg0201_38
- J1, TP10, TP11, TP12, TP5, TP6, TP7, TP8, TP9, U7: now not fitted; now left out of the parts list
- L1: footprint beeper-design:Pkg0201_2 -> beeper-design:Pkg0201_11
- L2: footprint beeper-design:Pkg0402_1 -> beeper-design:Pkg0402_5
- U1: footprint beeper-design:LP -> beeper-design:LP_7
Connections:
- net D+: now also U1.F1 (P2_10); no longer U1.F1 (P2_10)
- net D-: now also U1.G1 (P2_11); no longer U1.G1 (P2_11)
- net GND: now also U1.A11 (RFIOM2), U1.A12 (PSUBRF), U1.A8 (PSUB), U1.A9 (RFIOM1), U1.B9 (ESDN), U1.C12 (GND_RF2), U1.C2 (VSSIOQQ), U1.D12 (GND_RF1), U1.E11 (GND_XTAL2), U1.E12 (GND_XTAL1), U1.F5 (VSSD4), U1.F6 (VSSD3), U1.G12 (GND_XTAL3), U1.G5 (VSSD1), U1.G6 (VSSD2), U1.G7 (VSSD5), U1.H1 (GND_BOOST), U1.H6 (AVS1), U1.H7 (AVS2), U1.H8 (AVS3), U1.L8 (GND_SDADC), U1.L9 (GND_VAD), U1.M1 (GND_BUCK), C1.1, C11.1, C12.1, C2.1, C3.1, C4.1, C49.2, C5.1, C50.2, C6.1, C7.1, C8.1, C9.1; no longer U1.A11 (RFIOM2), U1.A12 (PSUBRF), U1.A8 (PSUB), U1.A9 (RFIOM1), U1.B9 (ESDN), U1.C12 (GND_RF2), U1.C2 (VSSIOQQ), U1.D12 (GND_RF1), U1.E11 (GND_XTAL2), U1.E12 (GND_XTAL1), U1.F5 (VSSD4), U1.F6 (VSSD3), U1.G12 (GND_XTAL3), U1.G5 (VSSD1), U1.G6 (VSSD2), U1.G7 (VSSD5), U1.H1 (GND_BOOST), U1.H6 (AVS1), U1.H7 (AVS2), U1.H8 (AVS3), U1.L8 (GND_SDADC), U1.L9 (GND_VAD), U1.M1 (GND_BUCK)
- net RF1: now also U1.A10 (RFIOP), C49.1, R11.1; no longer U1.A10 (RFIOP)
- net RF2: now also C50.1, R11.2, R19.1
- net RF3: now also R19.2
- net V18F: now also U1.C1 (V18F), C5.2, R1.1; no longer U1.C1 (V18F)
- net VBUS: now also U1.M5 (VBUS), C9.2; no longer U1.M5 (VBUS)
- net VDD1P8: now also U1.K2 (V18), C4.2; no longer U1.K2 (V18)
- net VDD1P8P: now also U1.J2 (V18P), C6.2, R1.2; no longer U1.J2 (V18P)
- net VDD3P0: now also U1.M6 (V30), C7.2; no longer U1.M6 (V30)
- net VDDSYS: now also U1.M3 (VSYS), C11.2, C12.2; no longer U1.M3 (VSYS)
- net VLED: now also U1.K1 (VLED); no longer U1.K1 (VLED)
- net at TP11.p: now also U1.M4 (VBAT), C8.2; no longer U1.M4 (VBAT)
- net at XTAL1.1: now also U1.F11 (XTAL32Mp); no longer U1.F11 (XTAL32Mp)
- net at XTAL1.3: now also U1.F12 (XTAL32Mm); no longer U1.F12 (XTAL32Mm)
- net at L2.1: now also U1.J1 (LZ); no longer U1.J1 (LZ)
- net at L1.2: now also U1.L1 (LY); no longer U1.L1 (LY)
- net at L1.1: now also U1.M2 (LX); no longer U1.M2 (LX)
- removed net board-io_b: U1.L4 (LED3)
- removed net board-io_g: U1.L6 (LED2)
- removed net board-io_r: U1.L5 (LED1)
- removed net mcu0_gpio: U1.D11 (P0_28)
- removed net mcu0_gpio1: U1.C10 (P0_11)
- removed net mcu0_gpio2: U1.E3 (P2_00)
- removed net mcu1_gpio: U1.E9 (P0_14)
- removed net mcu1_gpio1: U1.M8 (P1_06)
- removed net mcu1_gpio2: U1.E1 (P0_13)
- removed net mcu2_gpio: U1.D2 (P2_12)
- removed net mcu2_gpio1: U1.C4 (P0_26)
- removed net mcu3_gpio: U1.F2 (P1_28)
- net mcu_clk: no longer names the net of TP5.p
- net mcu_clk: now also U1.K5 (P0_31); no longer U1.K5 (P0_31)
- removed net mcu_cs: U1.H9 (P0_23)
- removed net mcu_cs1: U1.A6 (OQSIF_CS)
- net mcu_data0: no longer names the net of TP6.p
- net mcu_data0: now also U1.J8 (P1_30); no longer U1.J8 (P1_30)
- net mcu_data1: no longer names the net of TP7.p
- net mcu_data1: now also U1.K7 (P1_22); no longer U1.K7 (P1_22)
- net mcu_data2: no longer names the net of TP8.p
- net mcu_data2: now also U1.J7 (P1_31); no longer U1.J7 (P1_31)
- net mcu_data3: no longer names the net of TP9.p
- net mcu_data3: now also U1.K6 (P1_23); no longer U1.K6 (P1_23)
- net mcu_rx: no longer names the net of J1.3
- net mcu_rx: now also U1.H10 (P0_30); no longer U1.H10 (P0_30)
- removed net mcu_sck: U1.J9 (P2_01)
- removed net mcu_sck1: U1.B4 (OQSIF_CLK)
- removed net mcu_scl: U1.K9 (P1_12)
- removed net mcu_scl1: U1.E10 (P0_21)
- removed net mcu_scl2: U1.C3 (P0_25)
- removed net mcu_sda: U1.D4 (P0_12)
- removed net mcu_sda1: U1.C11 (P0_29)
- removed net mcu_sda2: U1.K8 (P1_11)
- removed net mcu_sdi: U1.M7 (P1_05)
- removed net mcu_sdio0: U1.A1 (OQSIF_D0)
- removed net mcu_sdio1: U1.A2 (OQSIF_D1)
- removed net mcu_sdio2: U1.A3 (OQSIF_D2)
- removed net mcu_sdio3: U1.B3 (OQSIF_D3)
- removed net mcu_sdo: U1.L7 (P0_27)
- net mcu_swdclk: no longer names the net of J1.4
- net mcu_swdclk: now also U1.D6 (P0_01); no longer U1.D6 (P0_01)
- net mcu_swdio: no longer names the net of J1.2
- net mcu_swdio: now also U1.C7 (P0_00); no longer U1.C7 (P0_00)
- net mcu_tx: no longer names the net of J1.6
- net mcu_tx: now also U1.B11 (P0_18); no longer U1.B11 (P0_18)
- new net: U1.J10 (NC), U1.J11 (NC), U1.J12 (NC), U1.K10 (NC), U1.K11 (NC), U1.K12 (NC), U1.L10 (NC), U1.L11 (NC), U1.L12 (NC), U1.M10 (NC), U1.M11 (NC), U1.M12 (NC)
- new net: C1.2, U1.L3 (V12)
- new net: C2.2, C3.2, U1.A7 (V14RF), U1.L2 (V14)
- new net board-io_rgb_b: U1.L4 (LED3)
- new net board-io_rgb_g: U1.L6 (LED2)
- new net board-io_rgb_r: U1.L5 (LED1)
- new net codec-i2c-net_scl: U1.C3 (P0_25)
- new net codec-i2c-net_sda: U1.D4 (P0_12)
- new net mcu_hap-gpio0_gpio: U1.D11 (P0_28)
- new net mcu_hap-gpio1_gpio: U1.E9 (P0_14)
- new net mcu_hap-i2c_scl: U1.E10 (P0_21)
- new net mcu_hap-i2c_sda: U1.C11 (P0_29)
- new net mcu_mcu-button0_gpio: U1.C10 (P0_11)
- new net mcu_mcu-button1_gpio: U1.M8 (P1_06)
- new net mcu_mcu-button2_gpio: U1.D2 (P2_12)
- new net mcu_mcu-mem_cs: U1.A6 (OQSIF_CS)
- new net mcu_mcu-mem_sck: U1.B4 (OQSIF_CLK)
- new net mcu_mcu-mem_sdio0: U1.A1 (OQSIF_D0)
- new net mcu_mcu-mem_sdio1: U1.A2 (OQSIF_D1)
- new net mcu_mcu-mem_sdio2: U1.A3 (OQSIF_D2)
- new net mcu_mcu-mem_sdio3: U1.B3 (OQSIF_D3)
- new net mcu_mcu-wpwr0_gpio: U1.E3 (P2_00)
- new net mcu_mcu-wpwr1_gpio: U1.E1 (P0_13)
- new net mcu_mcu-wpwr2_gpio: U1.C4 (P0_26)
- new net mcu_mcu-wpwr3_gpio: U1.F2 (P1_28)
- new net mcu_q-i3c_scl: U1.K9 (P1_12)
- new net mcu_q-i3c_sda: U1.K8 (P1_11)
- new net mcu_q-spi_cs: U1.H9 (P0_23)
- new net mcu_q-spi_sck: U1.J9 (P2_01)
- new net mcu_q-spi_sdi: U1.M7 (P1_05)
- new net mcu_q-spi_sdo: U1.L7 (P0_27)
- no-connect marks 3 -> 1
