File: designs/beeper-design/kicad/beeper-design-4.kicad_sch (KiCad schematic)
At the start: 7 parts, among them U12 DRV2605YZFR

Commit message: latest fully routed version
Parts:
- removed C47: 1u, beeper-design:Pkg0201_7, symbol my_capacitor_3
- removed C48: 1u, beeper-design:Pkg0201_14, symbol my_capacitor_7
- removed R16, R17: 8K2, beeper-design:Pkg0201_21, symbol my_resistor_3
- added C13: 1u, beeper-design:Pkg0201, symbol my_capacitor
- added C36: 100n, beeper-design:Pkg0201_2, symbol my_capacitor_1
- added C47: 1u, beeper-design:Pkg0201_27, symbol my_capacitor_15
- added C48: 1u, beeper-design:Pkg0201_37, symbol my_capacitor_21
- added J6: (no value), beeper-design:GCT_USB3100_XX_X_REVB_1, symbol component_2
- added R12, R13: 8K2, beeper-design:Pkg0201_1, symbol my_resistor
- added R14, R15: 8K2, beeper-design:Pkg0201_36, symbol my_resistor_12
- added R16, R17: 8K2, beeper-design:Pkg0201_5, symbol my_resistor_1
- added R18: 100K, beeper-design:Pkg0201_40, symbol my_resistor_14
- added U2: AT25FF321A-UUN-T, beeper-design:WLCSP_12, symbol AT25FF321A_UUN_T
- added U5: FH19C-6S-0.5SH(10), beeper-design:LP_3, symbol FH19C_6S_0_5SH_10_
- TP1, TP2: now not fitted; now left out of the parts list
- U12: footprint beeper-design:LP_7 -> beeper-design:LP_6
Connections:
- net GND: now also C13.1, C36.2, C47.1, C48.1, J6.5 (GND), R18.2, U2.C3 (GND), U5.2, U5.3, U5.4, U5.7, U5.8
- net VDDSYS: now also C48.2, R16.2, R17.2
- net at U12.A2 (REG): now also C47.2
- net mcu0_gpio renamed mcu_hap-gpio0_gpio
- net mcu1_gpio renamed mcu_hap-gpio1_gpio
- net mcu_scl1 renamed mcu_hap-i2c_scl
- net mcu_hap-i2c_scl: now also R17.1
- net mcu_sda1 renamed mcu_hap-i2c_sda
- net mcu_hap-i2c_sda: now also R16.1
- new net: U2.A1 (NC), U2.A5 (NC), U2.G1 (NC), U2.G5 (NC)
- new net D+: J6.3 (D+)
- new net D-: J6.2 (D-)
- new net MICBIAS1: U5.6
- new net SHIELD: C36.1, J6.6 (SHIELD), J6.7 (SHIELD), J6.8 (SHIELD), J6.9 (SHIELD), R18.1
- new net V18F: C13.2, U2.B2 (Vcc)
- new net VBUS: J6.1 (VBUS)
- new net VDD1P8: R14.2, R15.2
- new net VDD1P8P: R12.2, R13.2
- new net codec-i2c-net_scl: R13.1
- new net codec-i2c-net_sda: R12.1
- new net codec-pdm-net_clk: U5.1
- new net codec-pdm-net_data: U5.5
- new net mcu_mcu-mem_cs: U2.B4 (CSn)
- new net mcu_mcu-mem_sck: U2.F2 (SCK)
- new net mcu_mcu-mem_sdio0: U2.E3 (SI)
- new net mcu_mcu-mem_sdio1: U2.D4 (SO)
- new net mcu_mcu-mem_sdio2: U2.F4 (WPn)
- new net mcu_mcu-mem_sdio3: U2.D2 (HRn)
- new net mcu_q-i3c_scl: R15.1
- new net mcu_q-i3c_sda: R14.1
