File: designs/beeper-design/kicad/beeper-design-5.kicad_sch (KiCad schematic)
At the start: 24 parts, among them U3 BQ51003YFPR

Commit message: latest fully routed version
Parts:
- removed C15: 470n, beeper-design:Pkg0201_4, symbol my_capacitor_1
- removed C16: 470n, beeper-design:Pkg0201_11, symbol my_capacitor_5
- removed C19: 10n, beeper-design:Pkg0201_31, symbol my_capacitor_18
- removed C20: 10n, beeper-design:Pkg0201_40, symbol my_capacitor_22
- removed C21: 270p, beeper-design:Pkg0201_46, symbol my_capacitor_25
- removed C22: 10n, beeper-design:Pkg0201_3, symbol my_capacitor
- removed C23: 10u, beeper-design:Pkg0402_2, symbol C105225_1
- removed R2: 845R, beeper-design:Pkg0201_6, symbol my_resistor
- removed R20: 0R, beeper-design:Pkg0201_29, symbol my_resistor_7
- removed R21: 0R, beeper-design:Pkg0201_37, symbol my_resistor_10
- removed R3: 10K, beeper-design:Pkg0201_33, symbol my_resistor_9
- removed R4: 20K, beeper-design:Pkg0201_18, symbol my_resistor_2
- removed R5: 10K, beeper-design:Pkg0201_26, symbol my_resistor_5
- removed R7: 10K, beeper-design:Pkg0201_41, symbol my_resistor_13
- removed R8: 1K, beeper-design:Pkg0201_45, symbol my_resistor_15
- added C15: 470n, beeper-design:Pkg0201_42, symbol my_capacitor_24
- added C16: 470n, beeper-design:Pkg0201_4, symbol my_capacitor_3
- added C19: 10n, beeper-design:Pkg0201_41, symbol my_capacitor_23
- added C20: 10n, beeper-design:Pkg0201_3, symbol my_capacitor_2
- added C21: 270p, beeper-design:Pkg0201_16, symbol my_capacitor_9
- added C22: 10n, beeper-design:Pkg0201_28, symbol my_capacitor_16
- added C23: 10u, beeper-design:Pkg0402_8, symbol C105225_5
- added R2: 845R, beeper-design:Pkg0201_9, symbol my_resistor_4
- added R20: 0R, beeper-design:Pkg0201_15, symbol my_resistor_5
- added R21: 0R, beeper-design:Pkg0201_25, symbol my_resistor_9
- added R3: 10K, beeper-design:Pkg0201_6, symbol my_resistor_2
- added R4: 20K, beeper-design:Pkg0201_34, symbol my_resistor_11
- added R5: 10K, beeper-design:Pkg0201_44, symbol my_resistor_15
- added R7: 10K, beeper-design:Pkg0201_19, symbol my_resistor_7
- added R8: 1K, beeper-design:Pkg0201_31, symbol my_resistor_10
- C14: footprint beeper-design:Pkg0201_1 -> beeper-design:Pkg0201_45
- C17: footprint beeper-design:Pkg0201_17 -> beeper-design:Pkg0201_18
- C18: footprint beeper-design:Pkg0201_25 -> beeper-design:Pkg0201_30
- C24: footprint beeper-design:Pkg0402_5 -> beeper-design:Pkg0402_1
- C25: footprint beeper-design:Pkg0402_6 -> beeper-design:Pkg0402_3
- R6: footprint beeper-design:Pkg0201_13 -> beeper-design:Pkg0201_23
- TP13, TP14: now not fitted; now left out of the parts list
- U3: footprint beeper-design:LP_6 -> beeper-design:LP_5
Connections:
- net GND: now also C23.1, R3.2, R5.2, R7.2, R8.2
- net at C17.1, U3.B3 (AC1), U3.B4 (AC1): now also C15.1, C19.1, C21.2, C22.2
- net at U3.G3 (EN1): now also R20.1, R5.1
- net at C18.1, TP14.p, U3.B1 (AC2)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: now also C16.1, C20.1, C21.1
- net at R6.1, U3.F2 (FOD): now also R2.2, R4.1
- net at C24.2, U3.C2 (RECT), U3.C3 (RECT): now also C23.2, R4.2
- net at U3.C1 (BOOT2): now also C20.2
- net at U3.C4 (BOOT1): now also C19.2
- net at U3.E2 (CLAMP2): now also C16.2
- net at U3.E3 (CLAMP1): now also C15.2
- net at U3.G1 (ILIM): now also R2.1
- net at U3.G2 (EN2): now also R21.1, R3.1
- net at U3.G4 (AD): now also R8.1
- net at TP13.p: now also C22.1
- net mcu2_gpio1 renamed mcu_mcu-wpwr2_gpio
- net mcu3_gpio renamed mcu_mcu-wpwr3_gpio
- net mcu_mcu-wpwr3_gpio: now also R7.1
- new net mcu_mcu-wpwr0_gpio: R20.2
- new net mcu_mcu-wpwr1_gpio: R21.2
