File: designs/beeper-design/kicad/beeper-design.kicad_sch (KiCad schematic)
At the start: 0 parts

Commit message: exported to Kicad, fixed Kicad, exported gerbers
Changed lines of the file:
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@@
   (wire (pts (xy 200.66 128.27) (xy 200.66 121.92)) (stroke (width 0.127) (type default) (color 0 0 0 0)))
   (wire (pts (xy 245.11 106.68) (xy 245.11 100.33)) (stroke (width 0.127) (type default) (color 0 0 0 0)))
-  (wire (pts (xy 176.53 102.87) (xy 255.27 102.87)) (stroke (width 0.127) (type default) (color 0 0 0 0)))
-  (wire (pts (xy 251.46 132.08) (xy 255.27 132.08)) (stroke (width 0.127) (type default) (color 0 0 0 0)))
-  (wire (pts (xy 176.53 132.08) (xy 177.8 132.08)) (stroke (width 0.127) (type default) (color 0 0 0 0)))
-  (wire (pts (xy 255.27 132.08) (xy 255.27 102.87)) (stroke (width 0.127) (type default) (color 0 0 0 0)))
-  (wire (pts (xy 176.53 132.08) (xy 176.53 102.87)) (stroke (width 0.127) (type default) (color 0 0 0 0)))
-  (wire (pts (xy 234.95 138.43) (xy 238.76 138.43)) (stroke (width 0.127) (type default) (color 0 0 0 0)))
-  (wire (pts (xy 217.17 138.43) (xy 219.71 138.43)) (stroke (width 0.127) (type default) (color 0 0 0 0)))
-  (wire (pts (xy 219.71 128.27) (xy 234.95 128.27)) (stroke (width 0.127) (type default) (color 0 0 0 0)))
-  (wire (pts (xy 234.95 138.43) (xy 234.95 128.27)) (stroke (width 0.127) (type default) (color 0 0 0 0)))
-  (wire (pts (xy 219.71 138.43) (xy 219.71 128.27)) (stroke (width 0.127) (type default) (color 0 0 0 0)))
-  (wire (pts (xy 236.22 134.62) (xy 238.76 134.62)) (stroke (width 0.127) (type default) (color 0 0 0 0)))
-  (wire (pts (xy 233.68 135.89) (xy 236.22 135.89)) (stroke (width 0.127) (type default) (color 0 0 0 0)))
-  (wire (pts (xy 236.22 135.89) (xy 236.22 134.62)) (stroke (width 0.127) (type default) (color 0 0 0 0)))
+  (wire (pts (xy 176.53 138.43) (xy 177.8 138.43)) (stroke (width 0.127) (type default) (color 0 0 0 0)))
+  (wire (pts (xy 176.53 118.11) (xy 218.44 118.11)) (stroke (width 0.127) (type default) (color 0 0 0 0)))
+  (wire (pts (xy 217.17 132.08) (xy 218.44 132.08)) (stroke (width 0.127) (type default) (color 0 0 0 0)))
+  (wire (pts (xy 176.53 138.43) (xy 176.53 118.11)) (stroke (width 0.127) (type default) (color 0 0 0 0)))
+  (wire (pts (xy 218.44 132.08) (xy 218.44 118.11)) (stroke (width 0.127) (type default) (color 0 0 0 0)))
+  (wire (pts (xy 234.95 134.62) (xy 238.76 134.62)) (stroke (width 0.127) (type default) (color 0 0 0 0)))
+  (wire (pts (xy 233.68 135.89) (xy 234.95 135.89)) (stroke (width 0.127) (type default) (color 0 0 0 0)))
+  (wire (pts (xy 234.95 135.89) (xy 234.95 134.62)) (stroke (width 0.127) (type default) (color 0 0 0 0)))
   (wire (pts (xy 237.49 105.41) (xy 252.73 105.41)) (stroke (width 0.127) (type default) (color 0 0 0 0)))
   (wire (pts (xy 251.46 113.03) (xy 252.73 113.03)) (stroke (width 0.127) (type default) (color 0 0 0 0)))
@@
   (wire (pts (xy 252.73 113.03) (xy 252.73 105.41)) (stroke (width 0.127) (type default) (color 0 0 0 0)))
   (wire (pts (xy 237.49 130.81) (xy 237.49 105.41)) (stroke (width 0.127) (type default) (color 0 0 0 0)))
+  (wire (pts (xy 175.26 102.87) (xy 254.0 102.87)) (stroke (width 0.127) (type default) (color 0 0 0 0)))
+  (wire (pts (xy 251.46 132.08) (xy 254.0 132.08)) (stroke (width 0.127) (type default) (color 0 0 0 0)))
+  (wire (pts (xy 175.26 132.08) (xy 177.8 132.08)) (stroke (width 0.127) (type default) (color 0 0 0 0)))
+  (wire (pts (xy 254.0 132.08) (xy 254.0 102.87)) (stroke (width 0.127) (type default) (color 0 0 0 0)))
+  (wire (pts (xy 175.26 132.08) (xy 175.26 102.87)) (stroke (width 0.127) (type default) (color 0 0 0 0)))
   (wire (pts (xy 193.04 135.89) (xy 196.85 135.89)) (stroke (width 0.127) (type default) (color 0 0 0 0)))
-  (wire (pts (xy 251.46 138.43) (xy 254.0 138.43)) (stroke (width 0.127) (type default) (color 0 0 0 0)))
-  (wire (pts (xy 196.85 104.14) (xy 254.0 104.14)) (stroke (width 0.127) (type default) (color 0 0 0 0)))
+  (wire (pts (xy 251.46 138.43) (xy 255.27 138.43)) (stroke (width 0.127) (type default) (color 0 0 0 0)))
+  (wire (pts (xy 196.85 104.14) (xy 255.27 104.14)) (stroke (width 0.127) (type default) (color 0 0 0 0)))
   (wire (pts (xy 196.85 134.62) (xy 198.12 134.62)) (stroke (width 0.127) (type default) (color 0 0 0 0)))
-  (wire (pts (xy 254.0 138.43) (xy 254.0 104.14)) (stroke (width 0.127) (type default) (color 0 0 0 0)))
+  (wire (pts (xy 255.27 138.43) (xy 255.27 104.14)) (stroke (width 0.127) (type default) (color 0 0 0 0)))
   (wire (pts (xy 196.85 135.89) (xy 196.85 104.14)) (stroke (width 0.127) (type default) (color 0 0 0 0)))
-  (wire (pts (xy 175.26 138.43) (xy 177.8 138.43)) (stroke (width 0.127) (type default) (color 0 0 0 0)))
-  (wire (pts (xy 175.26 118.11) (xy 218.44 118.11)) (stroke (width 0.127) (type default) (color 0 0 0 0)))
-  (wire (pts (xy 217.17 132.08) (xy 218.44 132.08)) (stroke (width 0.127) (type default) (color 0 0 0 0)))
-  (wire (pts (xy 175.26 138.43) (xy 175.26 118.11)) (stroke (width 0.127) (type default) (color 0 0 0 0)))
-  (wire (pts (xy 218.44 132.08) (xy 218.44 118.11)) (stroke (width 0.127) (type default) (color 0 0 0 0)))
+  (wire (pts (xy 236.22 138.43) (xy 238.76 138.43)) (stroke (width 0.127) (type default) (color 0 0 0 0)))
+  (wire (pts (xy 217.17 138.43) (xy 219.71 138.43)) (stroke (width 0.127) (type default) (color 0 0 0 0)))
+  (wire (pts (xy 219.71 124.46) (xy 236.22 124.46)) (stroke (width 0.127) (type default) (color 0 0 0 0)))
+  (wire (pts (xy 236.22 138.43) (xy 236.22 124.46)) (stroke (width 0.127) (type default) (color 0 0 0 0)))
+  (wire (pts (xy 219.71 138.43) (xy 219.71 124.46)) (stroke (width 0.127) (type default) (color 0 0 0 0)))
 (junction (at 227.33 143.51) (diameter 0.762) (color 0 0 0 0 ))
 (junction (at 207.01 143.51) (diameter 0.762) (color 0 0 0 0 ))
@@
     (instances
       (project "beeper-design"
-        (path "/aa3cd5e6-b5a4-ca24-66fa-941455dab46f"
+        (path "/e5432c0b-b6b8-29a4-750f-8ef474db255b"
           (reference "#PWR?") (unit 1)
         )
@@
     (instances
       (project "beeper-design"
-        (path "/aa3cd5e6-b5a4-ca24-66fa-941455dab46f"
+        (path "/e5432c0b-b6b8-29a4-750f-8ef474db255b"
           (reference "#PWR?") (unit 1)
         )
@@
     (instances
       (project "beeper-design"
-        (path "/aa3cd5e6-b5a4-ca24-66fa-941455dab46f"
+        (path "/e5432c0b-b6b8-29a4-750f-8ef474db255b"
           (reference "#PWR?") (unit 1)
         )
@@
     (instances
       (project "beeper-design"
-        (path "/aa3cd5e6-b5a4-ca24-66fa-941455dab46f"
+        (path "/e5432c0b-b6b8-29a4-750f-8ef474db255b"
           (reference "#PWR?") (unit 1)
         )
@@
     (instances
       (project "beeper-design"
-        (path "/aa3cd5e6-b5a4-ca24-66fa-941455dab46f"
+        (path "/e5432c0b-b6b8-29a4-750f-8ef474db255b"
           (reference "#PWR?") (unit 1)
         )
@@
     (instances
       (project "beeper-design"
-        (path "/aa3cd5e6-b5a4-ca24-66fa-941455dab46f"
+        (path "/e5432c0b-b6b8-29a4-750f-8ef474db255b"
           (reference "#PWR?") (unit 1)
         )
@@
     (instances
       (project "beeper-design"
-        (path "/aa3cd5e6-b5a4-ca24-66fa-941455dab46f"
+        (path "/e5432c0b-b6b8-29a4-750f-8ef474db255b"
           (reference "#PWR?") (unit 1)
         )
@@
     (instances
       (project "beeper-design"
-        (path "/aa3cd5e6-b5a4-ca24-66fa-941455dab46f"
+        (path "/e5432c0b-b6b8-29a4-750f-8ef474db255b"
           (reference "#PWR?") (unit 1)
         )
@@
     (instances
       (project "beeper-design"
-        (path "/aa3cd5e6-b5a4-ca24-66fa-941455dab46f"
+        (path "/e5432c0b-b6b8-29a4-750f-8ef474db255b"
           (reference "#PWR?") (unit 1)
         )
@@
     (instances
       (project "beeper-design"
-        (path "/aa3cd5e6-b5a4-ca24-66fa-941455dab46f"
+        (path "/e5432c0b-b6b8-29a4-750f-8ef474db255b"
           (reference "#PWR?") (unit 1)
         )
@@
     (instances
       (project "beeper-design"
-        (path "/aa3cd5e6-b5a4-ca24-66fa-941455dab46f"
+        (path "/e5432c0b-b6b8-29a4-750f-8ef474db255b"
           (reference "#PWR?") (unit 1)
         )
@@
     (instances
       (project "beeper-design"
-        (path "/aa3cd5e6-b5a4-ca24-66fa-941455dab46f"
+        (path "/e5432c0b-b6b8-29a4-750f-8ef474db255b"
           (reference "#PWR?") (unit 1)
         )
@@
     (instances
       (project "beeper-design"
-        (path "/aa3cd5e6-b5a4-ca24-66fa-941455dab46f"
+        (path "/e5432c0b-b6b8-29a4-750f-8ef474db255b"
           (reference "#PWR?") (unit 1)
         )
@@
     (instances
       (project "beeper-design"
-        (path "/aa3cd5e6-b5a4-ca24-66fa-941455dab46f" (page "2"))
+        (path "/e5432c0b-b6b8-29a4-750f-8ef474db255b" (page "2"))
       )
     )
@@
     (instances
       (project "beeper-design"
-        (path "/aa3cd5e6-b5a4-ca24-66fa-941455dab46f" (page "3"))
+        (path "/e5432c0b-b6b8-29a4-750f-8ef474db255b" (page "3"))
       )
     )
@@
     (instances
       (project "beeper-design"
-        (path "/aa3cd5e6-b5a4-ca24-66fa-941455dab46f" (page "4"))
+        (path "/e5432c0b-b6b8-29a4-750f-8ef474db255b" (page "4"))
       )
     )
@@
     (instances
       (project "beeper-design"
-        (path "/aa3cd5e6-b5a4-ca24-66fa-941455dab46f" (page "5"))
+        (path "/e5432c0b-b6b8-29a4-750f-8ef474db255b" (page "5"))
       )
     )
@@
     (instances
       (project "beeper-design"
-        (path "/aa3cd5e6-b5a4-ca24-66fa-941455dab46f" (page "6"))
-      )
-    )
+        (path "/e5432c0b-b6b8-29a4-750f-8ef474db255b" (page "6"))
+      )
+    )

Commit message: latest fully routed version
Other:
- removed sheet 
- removed sheet board-io.hapdrv
- removed sheet board-io.rs flex-conn mcu
- added sheet board-io flex-conn mcu (beeper-design-4.kicad_sch)
- added sheet mcu (beeper-design-2.kicad_sch)
